Commit message: 取消轮电机在旋转方向的惯量，等效到joint的armature上，绕开”虚空阻尼“问题

File: model/Infantry_25/urdf/Infantry_25_headless.urdf (robot description, URDF)
Before this commit: robot Wheel-Legged-Infantry, 9 links, 8 joints
Links:
- removed link gimbal_pitch_link
- removed link gimbal_yaw_link
Joints:
- removed joint gimbal_pitch_joint
- removed joint gimbal_yaw_joint
- joint wheel_r_joint: limit effort=5 velocity=60 -> effort=100 velocity=60; type continuous -> revolute
